Commit message: update navigation on the first floor

File: src/jackal_description/urdf/jackal.urdf.xacro (robot description, xacro)
@@ -218,6 +218,49 @@
     <origin xyz="${mount_spacing} 0 0" />
   </joint>
+  <!-- Depth Camera Link -->
+	<link name="depth_camera_link">
+	  <visual>
+	    <geometry>
+	      <box size="0.05 0.05 0.05"/>
+	    </geometry>
+	    <material name="black"/>
+	  </visual>
+	</link>
+	<joint name="depth_camera_joint" type="fixed">
+	  <parent link="front_mount"/>
+	  <child link="depth_camera_link"/>
+	  <origin xyz="0.1 0 0.1" rpy="0 0 0"/>
+	</joint>
   <!-- Bring in simulation data for Gazebo. -->
   <xacro:include filename="$(find jackal_description)/urdf/jackal.gazebo" />
+  <!-- Depth Camera Gazebo Plugin -->
+<gazebo reference="depth_camera_link">
+  <sensor type="depth" name="depth_camera">
+    <update_rate>30</update_rate>
+    <camera>
+      <horizontal_fov>1.047</horizontal_fov>
+      <image>
+        <width>640</width>
+        <height>480</height>
+        <format>R8G8B8</format>
+      </image>
+      <clip>
+        <near>0.1</near>
+        <far>10.0</far>
+      </clip>
+    </camera>
+    <plugin name="depth_camera_controller" filename="libgazebo_ros_depth_camera.so">
+      <alwaysOn>true</alwaysOn>
+      <updateRate>30</updateRate>
+      <cameraName>front_depth</cameraName>
+      <imageTopicName>image_raw</imageTopicName>
+      <cameraInfoTopicName>camera_info</cameraInfoTopicName>
+      <depthImageTopicName>depth/image_raw</depthImageTopicName>
+      <pointCloudTopicName>points</pointCloudTopicName>
+      <frameName>depth_camera_link</frameName>
+      <hackBaseline>0.07</hackBaseline>
+    </plugin>
+  </sensor>
+</gazebo>
   <!-- Optional standard accessories, including their simulation data. The rendering
        of these into the final description is controlled by optenv variables, which
